File: hardware/core/desky-core.kicad_pcb (KiCad board)
At the start: 2 copper layers, 100 x 80 mm, 0 parts

Commit message: hardware milestone: hierarchy, receptacles, tcrt module + guides
Parts:
- added J1: S3-LEFT, Connector_PinHeader_2.54mm:PinHeader_1x22_P2.54mm_Vertical, F.Cu at (36.0, 8.00)
- added J2: S3-RIGHT, Connector_PinHeader_2.54mm:PinHeader_1x22_P2.54mm_Vertical, F.Cu at (64.0, 8.00)
- added J3: DRV-LOGIC, Connector_PinHeader_2.54mm:PinHeader_1x06_P2.54mm_Vertical, F.Cu at (86.0, 6.00)
- added J4: DRV-MOTOR, Connector_PinHeader_2.54mm:PinHeader_1x06_P2.54mm_Vertical, F.Cu at (86.0, 27.0)
- added J5: MOT-L, Connector_JST:JST_XH_S2B-XH-A_1x02_P2.50mm_Horizontal, F.Cu at (79.0, 52.0)
- added J6: MOT-R, Connector_JST:JST_XH_S2B-XH-A_1x02_P2.50mm_Horizontal, F.Cu at (89.0, 52.0)
- added J7: TOF-VL53L0X, Connector_JST:JST_XH_B4B-XH-A_1x04_P2.50mm_Vertical, F.Cu at (10.0, 8.00)
- added J8: MPU-6500, Connector_PinHeader_2.54mm:PinHeader_1x08_P2.54mm_Vertical, F.Cu at (10.0, 20.0)
- added J_AMP1: AMP-MAX98357A, Connector_PinHeader_2.54mm:PinHeader_1x07_P2.54mm_Vertical, F.Cu at (10.0, 45.0)
- added J_MICA1: MIC-L, Connector_PinHeader_2.54mm:PinHeader_1x06_P2.54mm_Vertical, F.Cu at (28.0, 44.0)
- added J_MICB1: MIC-R, Connector_PinHeader_2.54mm:PinHeader_1x06_P2.54mm_Vertical, F.Cu at (28.0, 64.0)
- added J_MODF1: MOD-FWD-RCPT, Connector_PinHeader_2.54mm:PinHeader_1x04_P2.54mm_Vertical, F.Cu at (10.0, 68.0)
- added J_MODR1: MOD-REV-RCPT, Connector_PinHeader_2.54mm:PinHeader_1x04_P2.54mm_Vertical, F.Cu at (20.0, 68.0)
- added J_PWR1: 5V-IN, Connector_JST:JST_XH_B2B-XH-A_1x02_P2.50mm_Vertical, F.Cu at (86.0, 70.0)
- added J_SA1: SERVO-ARM, Connector_PinHeader_2.54mm:PinHeader_1x03_P2.54mm_Vertical, F.Cu at (45.0, 69.0)
- added J_SH1: SERVO-HEAD, Connector_PinHeader_2.54mm:PinHeader_1x03_P2.54mm_Vertical, F.Cu at (57.0, 69.0)
