File: hardware/core/desky-core.kicad_sch (KiCad schematic)
At the start: 0 parts

Commit message: hardware milestone: hierarchy, receptacles, tcrt module + guides
Parts:
- added J1: S3-LEFT, Connector_PinHeader_2.54mm:PinHeader_1x22_P2.54mm_Vertical, symbol Connector:Conn_01x22_Socket
- added J2: S3-RIGHT, Connector_PinHeader_2.54mm:PinHeader_1x22_P2.54mm_Vertical, symbol Connector:Conn_01x22_Socket
- added J3: DRV-LOGIC, Connector_PinHeader_2.54mm:PinHeader_1x06_P2.54mm_Vertical, symbol Connector:Conn_01x06_Socket
- added J4: DRV-MOTOR, Connector_PinHeader_2.54mm:PinHeader_1x06_P2.54mm_Vertical, symbol Connector:Conn_01x06_Socket
- added J5: MOT-L, Connector_JST:JST_XH_S2B-XH-A_1x02_P2.50mm_Horizontal, symbol Connector:Conn_01x02_Socket
- added J6: MOT-R, Connector_JST:JST_XH_S2B-XH-A_1x02_P2.50mm_Horizontal, symbol Connector:Conn_01x02_Socket
- added J7: TOF-VL53L0X, Connector_JST:JST_XH_B4B-XH-A_1x04_P2.50mm_Vertical, symbol Connector:Conn_01x04_Socket
- added J8: MPU-6500, Connector_PinHeader_2.54mm:PinHeader_1x08_P2.54mm_Vertical, symbol Connector:Conn_01x08_Socket
- added J_AMP1: AMP-MAX98357A, Connector_PinHeader_2.54mm:PinHeader_1x07_P2.54mm_Vertical, symbol Connector:Conn_01x07_Socket
- added J_MICA1: MIC-L, Connector_PinHeader_2.54mm:PinHeader_1x06_P2.54mm_Vertical, symbol Connector:Conn_01x06_Socket
- added J_MICB1: MIC-R, Connector_PinHeader_2.54mm:PinHeader_1x06_P2.54mm_Vertical, symbol Connector:Conn_01x06_Socket
- added J_MODF1: MOD-FWD-RCPT, Connector_PinHeader_2.54mm:PinHeader_1x04_P2.54mm_Vertical, symbol Connector:Conn_01x04_Socket
- added J_MODR1: MOD-REV-RCPT, Connector_PinHeader_2.54mm:PinHeader_1x04_P2.54mm_Vertical, symbol Connector:Conn_01x04_Socket
- added J_PWR1: 5V-IN, Connector_JST:JST_XH_B2B-XH-A_1x02_P2.50mm_Vertical, symbol Connector:Conn_01x02_Socket
- added J_SA1: SERVO-ARM, Connector_PinHeader_2.54mm:PinHeader_1x03_P2.54mm_Vertical, symbol Connector:Conn_01x03_Socket
- added J_SH1: SERVO-HEAD, Connector_PinHeader_2.54mm:PinHeader_1x03_P2.54mm_Vertical, symbol Connector:Conn_01x03_Socket
Connections:
- new net EMIT_FWD: J1.19 (Pin_19), J_MODF1.4 (Pin_4)
- new net EMIT_REV: J1.20 (Pin_20), J_MODR1.4 (Pin_4)
- new net GND: J1.22 (Pin_22), J2.1 (Pin_1), J2.21 (Pin_21), J2.22 (Pin_22), J3.3 (Pin_3), J7.2 (Pin_2), J8.2 (Pin_2), J8.7 (Pin_7), J_AMP1.6 (Pin_6), J_MICA1.3 (Pin_3), J_MICA1.6 (Pin_6), J_MICB1.6 (Pin_6), J_MODF1.2 (Pin_2), J_MODR1.2 (Pin_2), J_PWR1.2 (Pin_2), J_SA1.3 (Pin_3), J_SH1.3 (Pin_3)
- new net I2C_SCL: J1.17 (Pin_17), J7.4 (Pin_4), J8.3 (Pin_3)
- new net I2C_SDA: J1.16 (Pin_16), J7.3 (Pin_3), J8.4 (Pin_4)
- new net I2S_BCLK: J1.9 (Pin_9), J_AMP1.2 (Pin_2), J_MICA1.1 (Pin_1), J_MICB1.1 (Pin_1)
- new net I2S_DIN: J1.11 (Pin_11), J_MICA1.4 (Pin_4), J_MICB1.4 (Pin_4)
- new net I2S_DOUT: J1.10 (Pin_10), J_AMP1.3 (Pin_3)
- new net I2S_WS: J1.8 (Pin_8), J_AMP1.1 (Pin_1), J_MICA1.2 (Pin_2), J_MICB1.2 (Pin_2)
- new net MOT_L1: J4.2 (Pin_2), J5.1 (Pin_1)
- new net MOT_L2: J4.3 (Pin_3), J5.2 (Pin_2)
- new net MOT_R1: J4.4 (Pin_4), J6.1 (Pin_1)
- new net MOT_R2: J4.5 (Pin_5), J6.2 (Pin_2)
- new net M_FAULT: J1.12 (Pin_12), J4.6 (Pin_6)
- new net M_IN1: J1.4 (Pin_4), J3.6 (Pin_6)
- new net M_IN2: J1.5 (Pin_5), J3.5 (Pin_5)
- new net M_IN3: J1.6 (Pin_6), J3.2 (Pin_2)
- new net M_IN4: J1.7 (Pin_7), J3.1 (Pin_1)
- new net SERVO_ARM: J2.6 (Pin_6), J_SA1.1 (Pin_1)
- new net SERVO_HEAD: J2.7 (Pin_7), J_SH1.1 (Pin_1)
- new net TCRT_FWD: J2.4 (Pin_4), J_MODF1.3 (Pin_3)
- new net TCRT_REV: J2.5 (Pin_5), J_MODR1.3 (Pin_3)
- new net VCC_3V3: J1.1 (Pin_1), J1.2 (Pin_2), J7.1 (Pin_1), J8.1 (Pin_1), J_MICA1.5 (Pin_5), J_MICB1.3 (Pin_3), J_MICB1.5 (Pin_5), J_MODF1.1 (Pin_1), J_MODR1.1 (Pin_1)
- new net VCC_5V: J1.21 (Pin_21), J3.4 (Pin_4), J4.1 (Pin_1), J_AMP1.7 (Pin_7), J_PWR1.1 (Pin_1), J_SA1.2 (Pin_2), J_SH1.2 (Pin_2)
- no-connect marks 0 -> 25
Other:
- added sheet TCRT-FWD (../tcrt/tcrt-module.kicad_sch)
- added sheet TCRT-REV (../tcrt/tcrt-module.kicad_sch)
