File: hardware/head/desky-head.kicad_pcb (KiCad board)
At the start: 2 copper layers, 100 x 80 mm, 0 parts

Commit message: hardware milestone: hierarchy, receptacles, tcrt module + guides
Parts:
- added J_CAML: CAM-LEFT, Connector_PinHeader_2.54mm:PinHeader_1x08_P2.54mm_Vertical, F.Cu at (36.0, 30.0)
- added J_CAMR: CAM-RIGHT, Connector_PinHeader_2.54mm:PinHeader_1x08_P2.54mm_Vertical, F.Cu at (64.0, 30.0)
- added J_HPWR: 5V-IN, Connector_JST:JST_XH_B2B-XH-A_1x02_P2.50mm_Vertical, F.Cu at (86.0, 55.0)
- added J_OLED: OLED-096, Connector_PinHeader_2.54mm:PinHeader_1x04_P2.54mm_Vertical, F.Cu at (86.0, 30.0)
