File: hardware/head/desky-head.kicad_sch (KiCad schematic)
At the start: 0 parts

Commit message: hardware milestone: hierarchy, receptacles, tcrt module + guides
Parts:
- added J_CAML1: CAM-LEFT, Connector_PinHeader_2.54mm:PinHeader_1x08_P2.54mm_Vertical, symbol Connector:Conn_01x08_Socket
- added J_CAMR1: CAM-RIGHT, Connector_PinHeader_2.54mm:PinHeader_1x08_P2.54mm_Vertical, symbol Connector:Conn_01x08_Socket
- added J_HPWR1: 5V-IN, Connector_JST:JST_XH_B2B-XH-A_1x02_P2.50mm_Vertical, symbol Connector:Conn_01x02_Socket
- added J_OLED1: OLED-096, Connector_PinHeader_2.54mm:PinHeader_1x04_P2.54mm_Vertical, symbol Connector:Conn_01x04_Socket
Connections:
- new net GND: J_CAML1.7 (Pin_7), J_CAMR1.4 (Pin_4), J_CAMR1.8 (Pin_8), J_HPWR1.2 (Pin_2), J_OLED1.1 (Pin_1)
- new net OLED_SCL: J_CAML1.4 (Pin_4), J_OLED1.3 (Pin_3)
- new net OLED_SDA: J_CAML1.3 (Pin_3), J_OLED1.4 (Pin_4)
- new net VCC_3V3: J_CAMR1.1 (Pin_1), J_OLED1.2 (Pin_2)
- new net VCC_5V: J_CAML1.8 (Pin_8), J_HPWR1.1 (Pin_1)
- no-connect marks 0 -> 9
